File: pcb/sigmar.kicad_pcb (KiCad board)
At the start: 2 copper layers, 53 parts, among them J1 USB_Micro-B_Molex-105017-0001, J2 TRRS-PJ-320A, SW1 Cherry-MX-LED-APA102, SW10 Cherry-MX-LED-APA102, SW11 Cherry-MX-LED-APA102, SW12 Cherry-MX-LED-APA102, SW13 Cherry-MX-LED-APA102, SW14 Cherry-MX-LED-APA102, SW15 Cherry-MX-LED-APA102, SW16 Cherry-MX-LED-APA102, SW17 Cherry-MX-LED-APA102, SW18 Cherry-MX-LED-APA102, SW19 Cherry-MX-LED-APA102, SW2 Cherry-MX-LED-APA102, SW20 Cherry-MX-LED-APA102, SW21 Cherry-MX-LED-APA102, SW22 Cherry-MX-LED-APA102, SW23 Cherry-MX-LED-APA102, SW24 Cherry-MX-LED-APA102, SW25 Cherry-MX-LED-APA102, SW3 Cherry-MX-LED-APA102, SW4 Cherry-MX-LED-APA102, SW5 Cherry-MX-LED-APA102, SW6 Cherry-MX-LED-APA102, SW7 Cherry-MX-LED-APA102, SW8 Cherry-MX-LED-APA102, SW9 Cherry-MX-LED-APA102, U1 TQFP-44_10x10mm_P0.8mm

Commit message: pcb design nearly finalized
Parts:
- added C1: 10uF, Capacitor_SMD:C_0805_2012Metric, B.Cu at (200.2, 61.8)
- added C10: 6pF, Capacitor_SMD:C_0805_2012Metric, B.Cu at (168.8, 115.8)
- added C11: 6pF, Capacitor_SMD:C_0805_2012Metric, B.Cu at (168.8, 107.8)
- added C2: 0.1uF, Capacitor_SMD:C_0805_2012Metric, B.Cu at (149.8, 99.1)
- added C3: 0.1uF, Capacitor_SMD:C_0805_2012Metric, B.Cu at (160.1, 98.3)
- added C4: 0.1uF, Capacitor_SMD:C_0805_2012Metric, B.Cu at (145.0, 105.3)
- added C5: 0.1uF, Capacitor_SMD:C_0805_2012Metric, B.Cu at (158.7, 117.2)
- added C6: 0.1uF, Capacitor_SMD:C_0805_2012Metric, B.Cu at (146.6, 113.6)
- added C7: 0.1uF, Capacitor_SMD:C_0805_2012Metric, B.Cu at (163.6, 107.4)
- added C8: 1uF, Capacitor_SMD:C_0805_2012Metric, B.Cu at (156.2, 99.8)
- added D26: D, Diode_SMD:D_MiniMELF, F.Cu at (145.8, 99.0)
- added D27: PRTR5V0U2X, Package_TO_SOT_SMD:SOT-143, B.Cu at (193.4, 56.4)
- added F1: 500mA, Fuse:Fuse_0805_2012Metric, B.Cu at (200.2, 58.7)
- added R1: 10K, Resistor_SMD:R_0805_2012Metric, B.Cu at (163.9, 103.8)
- added R2: 10K, Resistor_SMD:R_0805_2012Metric, B.Cu at (149.3, 117.1)
- added R3: 5.1K, Resistor_SMD:R_0805_2012Metric, B.Cu at (199.0, 55.4)
- added R4: 5.1K, Resistor_SMD:R_0805_2012Metric, B.Cu at (187.9, 55.4)
- added R5: 22, Resistor_SMD:R_0805_2012Metric, B.Cu at (187.1, 58.7)
- added R6: 22, Resistor_SMD:R_0805_2012Metric, B.Cu at (189.5, 60.3)
- added SW26: SW_Push, Local:LL3301NF065QG, B.Cu at (212.5, 111.8)
- added USB1: HRO-TYPE-C-31-M-12, Type-C:HRO-TYPE-C-31-M-12, B.Cu at (193.4, 44.3)
- added Y1: 16MHz, Crystal:Crystal_SMD_3225-4Pin_3.2x2.5mm, B.Cu at (168.8, 111.8)
- D1, D10, D11, D12, D13, D14, D15, D16, D17, D18, D19, D2, D20, D21, D22, D23, D24, D25, D3, D4, D5, D6, D7, D8, D9: moved to B.Cu
- J1: value USB_Micro-B_Molex-105017-0001 -> AudioJack4; footprint Connector_USB:USB_Micro-B_Molex-105017-0001 -> Local:TRRS-PJ-320A; moved to B.Cu
- J2: value TRRS-PJ-320A -> AVR-ISP-6; footprint Local:TRRS-PJ-320A -> Local:AVR-ISP-6; moved to B.Cu
- SW13: footprint Local:SW_Cherry_MX_RGB_R2L -> Local:SW_Cherry_MX_RGB_R2L_2U
- U1: value TQFP-44_10x10mm_P0.8mm -> ATmega32U4-AU
- moved J1 146.2 mm to (222.0, 73.7), turned to 90 degrees
- moved D24 142.0 mm to (181.5, 126.1), turned to 180 degrees
- moved D25 141.5 mm to (201.4, 133.2), turned to 180 degrees
- moved SW1 141.2 mm to (98.2, 71.0)
- moved SW11 141.2 mm to (174.4, 77.7)
- moved SW13 141.2 mm to (212.5, 87.2)
- moved SW14 141.2 mm to (98.2, 109.1)
- moved SW15 141.2 mm to (117.2, 104.3)
- moved SW18 141.2 mm to (174.4, 96.7)
- moved SW2 141.2 mm to (117.2, 66.2)
- moved SW23 141.2 mm to (164.8, 122.4)
- moved SW5 141.2 mm to (174.4, 58.6)
- moved SW7 141.2 mm to (98.2, 90.0)
- moved SW8 141.2 mm to (117.2, 85.3)
- moved SW10 141.2 mm to (155.3, 72.9)
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Connections:
- D1 pad 1: /ROW1 -> Net-(D1-Pad1)
- D1 pad 2: Net-(D1-Pad2) -> /COL1
- D10 pad 1: /ROW2 -> Net-(D10-Pad1)
- D10 pad 2: Net-(D10-Pad2) -> /COL4
- D11 pad 1: /ROW2 -> Net-(D11-Pad1)
- D11 pad 2: Net-(D11-Pad2) -> /COL5
- D12 pad 1: /ROW2 -> Net-(D12-Pad1)
- D12 pad 2: Net-(D12-Pad2) -> /COL6
- D13 pad 1: /ROW2 -> Net-(D13-Pad1)
- D13 pad 2: Net-(D13-Pad2) -> /COL7
- D14 pad 1: /ROW3 -> Net-(D14-Pad1)
- D14 pad 2: Net-(D14-Pad2) -> /COL1
- D15 pad 1: /ROW3 -> Net-(D15-Pad1)
- D15 pad 2: Net-(D15-Pad2) -> /COL2
- D16 pad 1: /ROW3 -> Net-(D16-Pad1)
- D16 pad 2: Net-(D16-Pad2) -> /COL3
- D17 pad 1: /ROW3 -> Net-(D17-Pad1)
- D17 pad 2: Net-(D17-Pad2) -> /COL4
- D18 pad 1: /ROW3 -> Net-(D18-Pad1)
- D18 pad 2: Net-(D18-Pad2) -> /COL5
- D19 pad 1: /ROW3 -> Net-(D19-Pad1)
- D19 pad 2: Net-(D19-Pad2) -> /COL6
- D2 pad 1: /ROW1 -> Net-(D2-Pad1)
- D2 pad 2: Net-(D2-Pad2) -> /COL2
- D20 pad 1: /ROW4 -> Net-(D20-Pad1)
- D20 pad 2: Net-(D20-Pad2) -> /COL1
- D21 pad 1: /ROW4 -> Net-(D21-Pad1)
- D21 pad 2: Net-(D21-Pad2) -> /COL2
- D22 pad 1: /ROW4 -> Net-(D22-Pad1)
- D22 pad 2: Net-(D22-Pad2) -> /COL3
- D23 pad 1: /ROW4 -> Net-(D23-Pad1)
- D23 pad 2: Net-(D23-Pad2) -> /COL5
- D24 pad 1: /ROW4 -> Net-(D24-Pad1)
- D24 pad 2: Net-(D24-Pad2) -> /COL6
- D25 pad 1: /ROW4 -> Net-(D25-Pad1)
- D25 pad 2: Net-(D25-Pad2) -> /COL7
- D3 pad 1: /ROW1 -> Net-(D3-Pad1)
- D3 pad 2: Net-(D3-Pad2) -> /COL3
- D4 pad 1: /ROW1 -> Net-(D4-Pad1)
- D4 pad 2: Net-(D4-Pad2) -> /COL4
- D5 pad 1: /ROW1 -> Net-(D5-Pad1)
- D5 pad 2: Net-(D5-Pad2) -> /COL5
- D6 pad 1: /ROW1 -> Net-(D6-Pad1)
- D6 pad 2: Net-(D6-Pad2) -> /COL6
- D7 pad 1: /ROW2 -> Net-(D7-Pad1)
- D7 pad 2: Net-(D7-Pad2) -> /COL1
- D8 pad 1: /ROW2 -> Net-(D8-Pad1)
- D8 pad 2: Net-(D8-Pad2) -> /COL2
- D9 pad 1: /ROW2 -> Net-(D9-Pad1)
- D9 pad 2: Net-(D9-Pad2) -> /COL3
- J2 pad 1: (no net) -> /MISO
- J2 pad 2: (no net) -> VCC
- J2 pad 3: (no net) -> /SCK
- J2 pad 4: (no net) -> /MOSI
- SW1 pad 1: /COL1 -> Net-(D1-Pad1)
- SW1 pad 2: Net-(D1-Pad2) -> /ROW1
- SW10 pad 1: /COL4 -> Net-(D10-Pad1)
- SW10 pad 2: Net-(D10-Pad2) -> /ROW2
- SW11 pad 1: /COL5 -> Net-(D11-Pad1)
- SW11 pad 2: Net-(D11-Pad2) -> /ROW2
- SW12 pad 1: /COL6 -> Net-(D12-Pad1)
- SW12 pad 2: Net-(D12-Pad2) -> /ROW2
- SW13 pad 1: /COL7 -> Net-(D13-Pad1)
- SW13 pad 2: Net-(D13-Pad2) -> /ROW2
- SW14 pad 1: /COL1 -> Net-(D14-Pad1)
- SW14 pad 2: Net-(D14-Pad2) -> /ROW3
- SW15 pad 1: /COL2 -> Net-(D15-Pad1)
- SW15 pad 2: Net-(D15-Pad2) -> /ROW3
- SW16 pad 1: /COL3 -> Net-(D16-Pad1)
- SW16 pad 2: Net-(D16-Pad2) -> /ROW3
- SW17 pad 1: /COL4 -> Net-(D17-Pad1)
- SW17 pad 2: Net-(D17-Pad2) -> /ROW3
- SW18 pad 1: /COL5 -> Net-(D18-Pad1)
- SW18 pad 2: Net-(D18-Pad2) -> /ROW3
- SW19 pad 1: /COL6 -> Net-(D19-Pad1)
- SW19 pad 2: Net-(D19-Pad2) -> /ROW3
- SW2 pad 1: /COL2 -> Net-(D2-Pad1)
- SW2 pad 2: Net-(D2-Pad2) -> /ROW1
- SW20 pad 1: /COL1 -> Net-(D20-Pad1)
- SW20 pad 2: Net-(D20-Pad2) -> /ROW4
- SW21 pad 1: /COL2 -> Net-(D21-Pad1)
- SW21 pad 2: Net-(D21-Pad2) -> /ROW4
- SW22 pad 1: /COL3 -> Net-(D22-Pad1)
- SW22 pad 2: Net-(D22-Pad2) -> /ROW4
- SW23 pad 1: /COL4 -> Net-(D23-Pad1)
- SW23 pad 2: Net-(D23-Pad2) -> /ROW4
- SW24 pad 1: /COL5 -> Net-(D24-Pad1)
- SW24 pad 2: Net-(D24-Pad2) -> /ROW4
- SW25 pad 1: /COL6 -> Net-(D25-Pad1)
- SW25 pad 2: Net-(D25-Pad2) -> /ROW4
- SW3 pad 1: /COL3 -> Net-(D3-Pad1)
- SW3 pad 2: Net-(D3-Pad2) -> /ROW1
- SW4 pad 1: /COL4 -> Net-(D4-Pad1)
- SW4 pad 2: Net-(D4-Pad2) -> /ROW1
- SW5 pad 1: /COL5 -> Net-(D5-Pad1)
- SW5 pad 2: Net-(D5-Pad2) -> /ROW1
- SW6 pad 1: /COL6 -> Net-(D6-Pad1)
- SW6 pad 2: Net-(D6-Pad2) -> /ROW1
- SW7 pad 1: /COL1 -> Net-(D7-Pad1)
- SW7 pad 2: Net-(D7-Pad2) -> /ROW2
- SW8 pad 1: /COL2 -> Net-(D8-Pad1)
- SW8 pad 2: Net-(D8-Pad2) -> /ROW2
- SW9 pad 1: /COL3 -> Net-(D9-Pad1)
- SW9 pad 2: Net-(D9-Pad2) -> /ROW2
- U1 pad 1: (no net) -> /COL4
- U1 pad 10: (no net) -> /MOSI
- U1 pad 11: (no net) -> /MISO
- U1 pad 12: (no net) -> Net-(U1-Pad12)
- U1 pad 13: (no net) -> /RESET
- U1 pad 14: (no net) -> VCC
- U1 pad 15: (no net) -> GND
- U1 pad 16: (no net) -> /XTAL2
- U1 pad 17: (no net) -> /XTAL1
- U1 pad 18: (no net) -> Net-(U1-Pad18)
- U1 pad 19: (no net) -> Net-(U1-Pad19)
- U1 pad 2: (no net) -> VBUS
- U1 pad 20: (no net) -> Net-(U1-Pad20)
- U1 pad 21: (no net) -> /LED_CKI
- U1 pad 22: (no net) -> /LED_SDI
- U1 pad 23: (no net) -> GND
- U1 pad 24: (no net) -> VCC
- U1 pad 25: (no net) -> Net-(U1-Pad25)
- U1 pad 26: (no net) -> Net-(U1-Pad26)
- U1 pad 27: (no net) -> /COL5
- U1 pad 28: (no net) -> /COL6
- U1 pad 29: (no net) -> /COL7
- U1 pad 3: (no net) -> /D-
- U1 pad 30: (no net) -> /ROW4
- U1 pad 31: (no net) -> Net-(U1-Pad31)
- U1 pad 32: (no net) -> Net-(U1-Pad32)
- U1 pad 33: (no net) -> Net-(R2-Pad1)
- U1 pad 34: (no net) -> VCC
- U1 pad 35: (no net) -> GND
- U1 pad 36: (no net) -> /COL1
- U1 pad 37: (no net) -> /COL2
- U1 pad 38: (no net) -> /COL3
- U1 pad 39: (no net) -> /ROW1
- U1 pad 4: (no net) -> /D+
- U1 pad 40: (no net) -> /ROW2
- U1 pad 41: (no net) -> /ROW3
- U1 pad 42: (no net) -> Net-(U1-Pad42)
- U1 pad 43: (no net) -> GND
- U1 pad 44: (no net) -> VCC
- U1 pad 5: (no net) -> GND
- U1 pad 6: (no net) -> Net-(C8-Pad2)
- U1 pad 7: (no net) -> VBUS
- U1 pad 8: (no net) -> Net-(U1-Pad8)
- U1 pad 9: (no net) -> /SCK
Routing:
- net /ROW2: track 0.00 -> 162.6 mm, vias 0 -> 1
- net /ROW1: track 0.00 -> 161.3 mm
- net /ROW3: track 0.00 -> 120.9 mm
- net /ROW4: track 0.00 -> 115.1 mm
- net /COL1: track 0.00 -> 109.3 mm, vias 0 -> 2
- net VBUS: track 0.00 -> 107.3 mm, vias 0 -> 2
- net /COL7: track 0.00 -> 104.5 mm, vias 0 -> 2
- net /COL2: track 0.00 -> 98.3 mm, vias 0 -> 2
- net /MOSI: track 0.00 -> 96.4 mm, vias 0 -> 1
- net /MISO: track 0.00 -> 94.6 mm, vias 0 -> 1
- net /COL6: track 0.00 -> 93.9 mm, vias 0 -> 2
- net /COL5: track 0.00 -> 91.1 mm, vias 0 -> 2
- net /LED_SDI: track 0.00 -> 85.7 mm, vias 0 -> 3
- net /LED_CKI: track 0.00 -> 83.9 mm, vias 0 -> 3
- net GND: track 0.00 -> 82.5 mm, vias 0 -> 26
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- added copper zone on B.Cu, net GND
- added copper zone on F.Cu, net VCC
Other:
- net class Power added: clearance 0.127, trace_width 0.3048, via_dia 0.6, via_drill 0.3

Commit message: pcb updates
Parts:
- added R7: 10K, Resistor_SMD:R_0805_2012Metric, B.Cu at (219.8, 78.6)
- added R8: 10K, Resistor_SMD:R_0805_2012Metric, B.Cu at (216.2, 78.6)
- moved C3 1.45 mm to (160.5, 99.7), turned to 0 degrees
Connections:
- net /USB_CC renamed Net-(R4-Pad1)
- net /USB_VBus renamed Net-(D27-Pad4)
- J1 pad R1: /MOSI -> /SCL
- J1 pad R2: /MISO -> /SDA
- U1 pad 18: Net-(U1-Pad18) -> /SCL
- U1 pad 19: Net-(U1-Pad19) -> /SDA
Routing:
- net /SDA: track 0.00 -> 91.7 mm, vias 0 -> 2
- net /SCL: track 0.00 -> 91.4 mm, vias 0 -> 2
- net /MISO: track 94.6 -> 62.9 mm
- net /MOSI: track 96.4 -> 65.8 mm
- net VCC: track 53.0 -> 25.7 mm, vias 3 -> 6
- net /COL2: track 98.3 -> 102.4 mm
- net /COL1: track 109.3 -> 113.0 mm
- net GND: track 82.5 -> 80.0 mm
- net VBUS: track 107.3 -> 105.7 mm
- net /COL5: track 91.1 -> 92.7 mm, vias 2 -> 4
- net /LED_SDI: track 85.7 -> 86.3 mm
- net /LED_CKI: track 83.9 -> 84.6 mm

Commit message: pcb left v1.2
Parts:
- moved C1 0.07 mm to (200.2, 61.8)
Routing:
- net /MISO: track 62.9 -> 61.8 mm
- net /COL7: track 104.5 -> 103.7 mm
- added copper zone on F.Cu, net (none)
Other:
- board outline added: 133.4 x 101.7 mm
- board text added: "sigmar"
- board text added: "v1.2"
