File: pcb/sigmar.kicad_pcb (KiCad board)
At the start: 2 copper layers, 133.4 x 101.7 mm, 77 parts, among them J1 AudioJack4, J2 AVR-ISP-6, SW1 Cherry-MX-LED-APA102, SW10 Cherry-MX-LED-APA102, SW11 Cherry-MX-LED-APA102, SW12 Cherry-MX-LED-APA102, SW13 Cherry-MX-LED-APA102, SW14 Cherry-MX-LED-APA102, SW15 Cherry-MX-LED-APA102, SW16 Cherry-MX-LED-APA102, SW17 Cherry-MX-LED-APA102, SW18 Cherry-MX-LED-APA102, SW19 Cherry-MX-LED-APA102, SW2 Cherry-MX-LED-APA102, SW20 Cherry-MX-LED-APA102, SW21 Cherry-MX-LED-APA102, SW22 Cherry-MX-LED-APA102, SW23 Cherry-MX-LED-APA102, SW24 Cherry-MX-LED-APA102, SW25 Cherry-MX-LED-APA102, SW26 SW_Push, SW3 Cherry-MX-LED-APA102, SW4 Cherry-MX-LED-APA102, SW5 Cherry-MX-LED-APA102, SW6 Cherry-MX-LED-APA102, SW7 Cherry-MX-LED-APA102, SW8 Cherry-MX-LED-APA102, SW9 Cherry-MX-LED-APA102, U1 ATmega32U4-AU, Y1 16MHz

Commit message: fine tuning traces
Parts:
- moved R5 0.96 mm to (187.2, 59.7)
- moved R6 0.64 mm to (189.5, 59.7)
Routing:
- net /D+: track 62.4 -> 63.8 mm
- net /D-: track 64.7 -> 63.8 mm
- net /USB_D+: track 13.7 -> 12.9 mm
- net /USB_D-: track 11.7 -> 12.5 mm

Commit message: adjust
Parts:
- J2: value AVR-ISP-6 -> Reset_Pretty-Mask
- moved J1 3.28 mm to (224.9, 72.1)
Routing:
- net /SDA: track 91.7 -> 94.5 mm
- net /SCL: track 91.4 -> 93.1 mm
Other:
- board size 133.4 x 101.7 mm -> 136.2 x 101.7 mm
- board text added: "JLCJLCJLCJLC"

Commit message: pcb fixes
Parts:
- D1, D10, D11, D12, D13, D14, D15, D16, D17, D18, D19, D2, D20, D21, D22, D23, D24, D25, D3, D4, D5, D6, D7, D8, D9: footprint Diode_SMD:D_0805_2012Metric -> Diode_SMD:D_MiniMELF
- J2: value Reset_Pretty-Mask -> AVR-ISP-6
- moved D1 5.49 mm to (93.6, 73.4)
- moved D25 1.28 mm to (200.2, 133.9)
- moved D6 1.28 mm to (188.8, 71.0)
- moved D24 1.04 mm to (180.7, 126.7)
- moved J1 0.94 mm to (225.8, 71.9)
- moved D18 0.40 mm to (169.8, 99.1)
- moved D10 0.40 mm to (150.7, 75.3)
- moved D16 0.40 mm to (131.7, 99.1)
- moved D22 0.40 mm to (141.2, 124.8)
- moved D11 0.40 mm to (169.8, 80.0)
- moved D13 0.40 mm to (207.9, 89.6)
- moved D3 0.40 mm to (131.7, 61.0)
- moved D14 0.40 mm to (93.6, 111.5)
- moved D15 0.40 mm to (112.6, 106.7)
- moved D2 0.40 mm to (112.6, 68.6)
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Connections:
- net /USB_D+ renamed /components/USB_D+
- net /USB_D- renamed /components/USB_D-
- SW25 pad 6: Net-(SW25-Pad6) -> (no net)
- SW25 pad 7: Net-(SW25-Pad7) -> (no net)
- U1 pad 12: Net-(U1-Pad12) -> (no net)
- U1 pad 20: Net-(U1-Pad20) -> (no net)
- U1 pad 25: Net-(U1-Pad25) -> (no net)
- U1 pad 26: Net-(U1-Pad26) -> (no net)
- U1 pad 31: Net-(U1-Pad31) -> (no net)
- U1 pad 32: Net-(U1-Pad32) -> (no net)
- U1 pad 42: Net-(U1-Pad42) -> (no net)
- U1 pad 8: Net-(U1-Pad8) -> (no net)
- USB1 pad 3: Net-(USB1-Pad3) -> (no net)
- USB1 pad 9: Net-(USB1-Pad9) -> (no net)
Routing:
- net /COL4: track 57.8 -> 49.3 mm
- net /COL2: track 102.4 -> 95.0 mm
- net /COL5: track 92.7 -> 87.5 mm
- net /COL6: track 93.9 -> 96.1 mm
- net Net-(D6-Pad1): track 3.85 -> 2.67 mm
- net /COL1: track 113.0 -> 114.0 mm
- net Net-(D25-Pad1): track 3.82 -> 3.06 mm
- net Net-(D23-Pad1): track 3.50 -> 2.79 mm
- net Net-(D17-Pad1): track 3.50 -> 2.79 mm
- net Net-(D4-Pad1): track 3.50 -> 2.79 mm
- net Net-(D5-Pad1): track 3.50 -> 2.79 mm
- net Net-(D22-Pad1): track 3.50 -> 2.83 mm
- net Net-(D16-Pad1): track 3.50 -> 2.83 mm
- net Net-(D10-Pad1): track 3.50 -> 2.83 mm
- net Net-(D3-Pad1): track 3.50 -> 2.83 mm
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Other:
- board size 136.2 x 101.7 mm -> 137.1 x 101.7 mm
