File: pcb/sigmar.kicad_pcb (KiCad board)
At the start: 2 copper layers, 139.1 x 105.4 mm, 98 parts, among them J1 AudioJack4, J2 AVR-ISP-6, SW1 SW_Push_45deg, SW10 SW_Push_45deg, SW11 SW_Push_45deg, SW12 SW_Push_45deg, SW13 SW_Push_45deg, SW14 SW_Push_45deg, SW15 SW_Push_45deg, SW16 SW_Push_45deg, SW17 SW_Push_45deg, SW18 SW_Push_45deg, SW19 SW_Push_45deg, SW2 SW_Push_45deg, SW20 Rotary_Encoder_Switch, SW21 SW_Push_45deg, SW22 SW_Push_45deg, SW23 SW_Push_45deg, SW24 SW_Push_45deg, SW25 SW_Push_45deg, SW26 SW_Push_45deg, SW27 SW_Push, SW3 SW_Push_45deg, SW4 SW_Push_45deg, SW5 SW_Push_45deg, SW6 SW_Push_45deg, SW7 SW_Push_45deg, SW8 SW_Push_45deg, SW9 SW_Push_45deg, U1 Elite-C-V4

Commit message: pcb v1.3 final
Parts:
- moved D55 23.8 mm to (104.8, 79.5)
- moved D54 19.8 mm to (129.1, 71.9)
- moved D52 19.6 mm to (181.0, 76.7)
- moved D53 19.1 mm to (157.2, 71.9)
- moved D3 5.87 mm to (122.2, 70.0)
- moved D2 2.54 mm to (111.6, 77.6)
- moved D6 2.38 mm to (187.6, 74.8)
Routing:
- net Net-(D55-Pad2): track 78.2 -> 55.6 mm, vias 5 -> 6
- net Net-(D52-Pad2): track 48.2 -> 26.6 mm, vias 3 -> 2
- net Net-(D54-Pad2): track 46.6 -> 28.2 mm, vias 4 -> 2
- net COL3: track 74.9 -> 89.3 mm
- net Net-(D53-Pad2): track 43.4 -> 32.4 mm, vias 3 -> 4
- net LED: track 67.2 -> 57.4 mm, vias 1 -> 3
- net Net-(D31-Pad4): track 25.1 -> 20.0 mm
- net GND: track 59.9 -> 55.0 mm, vias 31 -> 34
- net Net-(D3-Pad1): track 6.08 -> 10.2 mm
- net ENC_A: track 118.5 -> 122.1 mm
- net ENC_B: track 124.8 -> 128.1 mm, vias 3 -> 5
- net +5V: track 55.1 -> 53.0 mm, vias 29 -> 32
- net Net-(D2-Pad1): track 6.08 -> 7.13 mm
- net Net-(D6-Pad1): track 6.08 -> 7.07 mm
- net COL2: track 96.2 -> 95.2 mm
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Other:
- outline, holes or cut-outs redrawn
