File: pcb/matrix.sch (KiCad schematic (older format))
At the start: 50 parts, among them SW1 Cherry-MX-LED-APA102, SW10 Cherry-MX-LED-APA102, SW11 Cherry-MX-LED-APA102, SW12 Cherry-MX-LED-APA102, SW13 Cherry-MX-LED-APA102, SW14 Cherry-MX-LED-APA102, SW15 Cherry-MX-LED-APA102, SW16 Cherry-MX-LED-APA102, SW17 Cherry-MX-LED-APA102, SW18 Cherry-MX-LED-APA102, SW19 Cherry-MX-LED-APA102, SW2 Cherry-MX-LED-APA102, SW20 Cherry-MX-LED-APA102, SW21 Cherry-MX-LED-APA102, SW22 Cherry-MX-LED-APA102, SW23 Cherry-MX-LED-APA102, SW24 Cherry-MX-LED-APA102, SW25 Cherry-MX-LED-APA102, SW3 Cherry-MX-LED-APA102, SW4 Cherry-MX-LED-APA102, SW5 Cherry-MX-LED-APA102, SW6 Cherry-MX-LED-APA102, SW7 Cherry-MX-LED-APA102, SW8 Cherry-MX-LED-APA102, SW9 Cherry-MX-LED-APA102

Commit message: pcb left v1.2
Connections:
- no-connect marks 0 -> 2
Changed lines of the file:
@@
 	11100 5950 11100 5850
 Connection ~ 11050 5950
+NoConn ~ 10100 5600
+NoConn ~ 10100 5700
 $EndSCHEMATC

Commit message: pcb fixes
Parts:
- SW13: footprint Local:SW_Cherry_MX_RGB_R2L -> Local:SW_Cherry_MX_RGB_R2L_2U
- SW7: footprint Local:SW_Cherry_MX_RGB_R2L -> Local:SW_Cherry_MX_RGB_L2R
Changed lines of the file:
@@
 $Descr A4 11693 8268
 encoding utf-8
-Sheet 2 2
+Sheet 2 3
 Title ""
 Date ""
@@
 F 0 "SW13" H 10475 3175 50  0000 C CNN
 F 1 "Cherry-MX-LED-APA102" H 10475 3084 50  0000 C CNN
-F 2 "Local:SW_Cherry_MX_RGB_R2L" H 10450 2300 50  0001 L TNN
+F 2 "Local:SW_Cherry_MX_RGB_R2L_2U" H 10450 2300 50  0001 L TNN
 F 3 "http://www.led-color.com/upload/201604/APA102-2020%20SMD%20LED.pdf" H 10500 2175 50  0001 L TNN
 	1    10400 2550
@@
 F 0 "SW7" H 1475 3175 50  0000 C CNN
 F 1 "Cherry-MX-LED-APA102" H 1475 3084 50  0000 C CNN
-F 2 "Local:SW_Cherry_MX_RGB_R2L" H 1450 2300 50  0001 L TNN
+F 2 "Local:SW_Cherry_MX_RGB_L2R" H 1450 2300 50  0001 L TNN
 F 3 "http://www.led-color.com/upload/201604/APA102-2020%20SMD%20LED.pdf" H 1500 2175 50  0001 L TNN
 	1    1400 2550
