File: pcb/sigmar.sch (KiCad schematic (older format))
At the start: 67 parts, among them SW1 Cherry-MX-LED-APA102, SW10 Cherry-MX-LED-APA102, SW11 Cherry-MX-LED-APA102, SW12 Cherry-MX-LED-APA102, SW13 Cherry-MX-LED-APA102, SW14 Cherry-MX-LED-APA102, SW15 Cherry-MX-LED-APA102, SW16 Cherry-MX-LED-APA102, SW17 Cherry-MX-LED-APA102, SW18 Cherry-MX-LED-APA102, SW19 Cherry-MX-LED-APA102, SW2 Cherry-MX-LED-APA102, SW20 Cherry-MX-LED-APA102, SW21 Cherry-MX-LED-APA102, SW22 Cherry-MX-LED-APA102, SW23 Cherry-MX-LED-APA102, SW24 Cherry-MX-LED-APA102, SW25 Cherry-MX-LED-APA102, SW3 Cherry-MX-LED-APA102, SW4 Cherry-MX-LED-APA102, SW5 Cherry-MX-LED-APA102, SW6 Cherry-MX-LED-APA102, SW7 Cherry-MX-LED-APA102, SW8 Cherry-MX-LED-APA102, SW9 Cherry-MX-LED-APA102, U1 ATmega32U4-AU

Commit message: pcb design nearly finalized
Parts:
- removed C? (x2): 0.1uF, symbol Device:C_Small
- removed C?: 1uF, symbol Device:CP1_Small
- removed C?: 10uF, symbol Device:CP1_Small
- removed D1, D10, D11, D12, D13, D14, D15, D16, D17, D18, D19, D2, D20, D21, D22, D23, D24, D25, D3, D4, D5, D6, D7, D8, D9: D, Diode_SMD:D_0805_2012Metric, symbol Device:D
- removed J?: USB_B_Micro, Connector_USB:USB_Micro-B_Molex-105017-0001, symbol Connector:USB_B_Micro
- removed SW1, SW13, SW14, SW15, SW16, SW17, SW18, SW19, SW2, SW3, SW4, SW5, SW6, SW7: Cherry-MX-LED-APA102, Local:SW_Cherry_MX_RGB_R2L, symbol Local:Cherry-MX-LED-APA102
- removed SW10, SW11, SW12, SW20, SW21, SW22, SW23, SW24, SW25, SW8, SW9: Cherry-MX-LED-APA102, Local:SW_Cherry_MX_RGB_L2R, symbol Local:Cherry-MX-LED-APA102
- added C1: 10uF, Capacitor_SMD:C_0805_2012Metric, symbol Device:C_Small
- added C2, C3, C6, C7: 0.1uF, Capacitor_SMD:C_0805_2012Metric, symbol Device:C_Small
- added C8: 1uF, Capacitor_SMD:C_0805_2012Metric, symbol Device:C_Small
- added D27: PRTR5V0U2X, Package_TO_SOT_SMD:SOT-143, symbol Power_Protection:PRTR5V0U2X
- added F1: 500mA, Fuse:Fuse_0805_2012Metric, symbol Device:Polyfuse_Small
- added J2: AVR-ISP-6, Local:AVR-ISP-6, symbol Connector:AVR-ISP-6
- added R2: 10K, Resistor_SMD:R_0805_2012Metric, symbol Device:R_Small
- added R3, R4: 5.1K, Resistor_SMD:R_0805_2012Metric, symbol Device:R_Small
- added USB1: HRO-TYPE-C-31-M-12, Type-C:HRO-TYPE-C-31-M-12, symbol Type-C:HRO-TYPE-C-31-M-12
- C10, C11, C4, C5: renamed from C?; footprint (none) -> Capacitor_SMD:C_0805_2012Metric
- D26: renamed from D?; footprint (none) -> Diode_SMD:D_MiniMELF
- R1: renamed from R?; value R_Small -> 10K; footprint (none) -> Resistor_SMD:R_0805_2012Metric
- R5, R6: renamed from R?; footprint (none) -> Resistor_SMD:R_0805_2012Metric
- SW26: renamed from SW?; footprint (none) -> Local:LL3301NF065QG
- Y1: renamed from Y?; footprint (none) -> Crystal:Crystal_SMD_3225-4Pin_3.2x2.5mm
- gave numbers to parts that had none: 1
Connections:
- net COL1: now also U1.36 (PF7)
- net COL2: now also U1.37 (PF6)
- net COL3: now also U1.38 (PF5)
- net COL4: now also U1.1 (PE6)
- net COL5: now also U1.27 (PD7)
- net COL6: now also U1.28 (PB4)
- net COL7: now also U1.29 (PB5)
- net GND: now also J1.S, C1.2, C2.2, C3.2, C6.2, C7.2, C8.1, D27.1 (GND), J2.6 (GND), R2.2, R3.1, R4.2, USB1.1 (GND), USB1.12 (GND), USB1.13 (SHIELD)
- net LED_CKI: now also U1.21 (PD3)
- net LED_SDI: now also U1.22 (PD5)
- net RESET: now also J2.5 (~RST)
- net ROW1: now also U1.39 (PF4)
- net ROW2: now also U1.40 (PF1)
- net ROW3: now also U1.41 (PF0)
- net ROW4: now also U1.30 (PB6)
- net VBUS: now also C1.1, C2.1, C3.1, F1.1
- net VCC: now also J1.T, C6.1, C7.1, J2.2 (VCC)
- net MOSI: now reaches U1.10 (PB2)
- net MOSI: now also J1.R1, J2.4 (MOSI)
- net MISO: now reaches U1.11 (PB3)
- net MISO: now also J1.R2, J2.1 (MISO)
- net XTAL2: now reaches C11.1, U1.16 (XTAL2), Y1.3
- net XTAL1: now reaches C10.1, U1.17 (XTAL1), Y1.1
- net D+: now reaches R6.1
- net D+: now also U1.4 (D+); no longer U1.3 (D-)
- net at U1.33 (~HWB~/PE2): now also R2.1
- net D-: now reaches R5.1
- net D-: now also U1.3 (D-); no longer U1.4 (D+)
- net at U1.6 (UCAP): now also C8.2
- net SCK: now reaches U1.9 (PB1)
- net SCK: now also J2.3 (SCK)
- net USB_D+: now reaches R6.2
- net USB_D+: now also D27.3 (I/O2), USB1.6 (DP1), USB1.8 (DP2)
- net USB_D-: now reaches R5.2
- net USB_D-: now also D27.2 (I/O1), USB1.5 (DN2), USB1.7 (DN1)
- new net: R3.2, USB1.10 (CC2)
- new net USB_CC: R4.1, USB1.4 (CC1)
- new net USB_VBus: D27.4 (VCC), F1.2, USB1.11 (VBUS), USB1.2 (VBUS)
Other:
- moved on the sheet: C10, C11, C4, C5, D26, J1, R1, R5, R6, SW26, U1, Y1

Commit message: pcb updates
Parts:
- added R? (x2): 10K, Resistor_SMD:R_0805_2012Metric, symbol Device:R_Small
Connections:
- net MISO: no longer J1.R2
- net MOSI: no longer J1.R1
- net VCC: now also R?.1, R?.1
- net SCL: now reaches U1.18 (PD0)
- net SCL: now also J1.R1, R?.2
- net SDA: now reaches U1.19 (PD1)
- net SDA: now also J1.R2, R?.2
- net USB_CC: no longer names the net of R4.1, USB1.4 (CC1)
- net USB_VBus: no longer names the net of D27.4 (VCC), F1.2, USB1.11 (VBUS), USB1.2 (VBUS)
Other:
- moved on the sheet: J1
Changed lines of the file:
@@
 L Connector:AudioJack4 J1
 U 1 1 60DE9A39
-P 8950 1650
-F 0 "J1" H 8907 1975 50  0000 C CNN
-F 1 "AudioJack4" H 8907 1884 50  0000 C CNN
-F 2 "Local:TRRS-PJ-320A" H 8950 1650 50  0001 C CNN
-F 3 "~" H 8950 1650 50  0001 C CNN
-	1    8950 1650
+P 9600 1650
+F 0 "J1" H 9557 1975 50  0000 C CNN
+F 1 "AudioJack4" H 9557 1884 50  0000 C CNN
+F 2 "Local:TRRS-PJ-320A" H 9600 1650 50  0001 C CNN
+F 3 "~" H 9600 1650 50  0001 C CNN
+	1    9600 1650
 	-1   0    0    1
 $EndComp
@@
 Text Label 7950 5450 0    50   ~ 0
 USB_D+
-Text Label 7950 4850 0    50   ~ 0
-USB_VBus
-Text Label 7550 5050 0    50   ~ 0
-USB_CC
 $Comp
 L power:GND #PWR0120
 U 1 1 61F4FC92
-P 8650 1850
-F 0 "#PWR0120" H 8650 1600 50  0001 C CNN
-F 1 "GND" H 8655 1677 50  0000 C CNN
-F 2 "" H 8650 1850 50  0001 C CNN
-F 3 "" H 8650 1850 50  0001 C CNN
-	1    8650 1850
-	1    0    0    -1
-$EndComp
-Wire Wire Line
-	8750 1750 8650 1750
-Wire Wire Line
-	8650 1750 8650 1850
-Wire Wire Line
-	8750 1450 8650 1450
-Wire Wire Line
-	8650 1450 8650 1350
+P 9300 1850
+F 0 "#PWR0120" H 9300 1600 50  0001 C CNN
+F 1 "GND" H 9305 1677 50  0000 C CNN
+F 2 "" H 9300 1850 50  0001 C CNN
+F 3 "" H 9300 1850 50  0001 C CNN
+	1    9300 1850
+	1    0    0    -1
+$EndComp
+Wire Wire Line
+	9400 1750 9300 1750
+Wire Wire Line
+	9300 1750 9300 1850
+Wire Wire Line
+	9400 1450 9300 1450
+Wire Wire Line
+	9300 1450 9300 1350
 $Comp
 L power:VCC #PWR0121
 U 1 1 61F590C6
-P 8650 1350
-F 0 "#PWR0121" H 8650 1200 50  0001 C CNN
-F 1 "VCC" H 8665 1523 50  0000 C CNN
-F 2 "" H 8650 1350 50  0001 C CNN
-F 3 "" H 8650 1350 50  0001 C CNN
-	1    8650 1350
-	1    0    0    -1
-$EndComp
-Wire Wire Line
-	8750 1550 8300 1550
-Wire Wire Line
-	8750 1650 8300 1650
+P 9300 1350
+F 0 "#PWR0121" H 9300 1200 50  0001 C CNN
+F 1 "VCC" H 9315 1523 50  0000 C CNN
+F 2 "" H 9300 1350 50  0001 C CNN
+F 3 "" H 9300 1350 50  0001 C CNN
+	1    9300 1350
+	1    0    0    -1
+$EndComp
+Wire Wire Line
+	9400 1550 9050 1550
 Text Label 3100 5700 0    50   ~ 0
 COL4
@@
 Text Label 3100 5000 0    50   ~ 0
 LED_CKI
-Text Label 8300 1650 0    50   ~ 0
-MISO
-Text Label 8300 1550 0    50   ~ 0
-MOSI
+Text Label 8500 1650 0    50   ~ 0
+SDA
+Text Label 8500 1550 0    50   ~ 0
+SCL
 Text Label 3100 4100 0    50   ~ 0
 ROW4
@@
 Text Label 3100 5400 0    50   ~ 0
 COL5
+Text Label 3100 4700 0    50   ~ 0
+SCL
+Text Label 3100 4800 0    50   ~ 0
+SDA
+$Comp
+L Device:R_Small R?
+U 1 1 6210052B
+P 9050 1350
+F 0 "R?" H 9109 1396 50  0000 L CNN
+F 1 "10K" H 9109 1305 50  0000 L CNN
+F 2 "Resistor_SMD:R_0805_2012Metric" H 9050 1350 50  0001 C CNN
+F 3 "~" H 9050 1350 50  0001 C CNN
+	1    9050 1350
+	1    0    0    -1
+$EndComp
+Connection ~ 9050 1550
+$Comp
+L Device:R_Small R?
+U 1 1 621066F7
+P 8800 1350
+F 0 "R?" H 8859 1396 50  0000 L CNN
+F 1 "10K" H 8859 1305 50  0000 L CNN
+F 2 "Resistor_SMD:R_0805_2012Metric" H 8800 1350 50  0001 C CNN
+F 3 "~" H 8800 1350 50  0001 C CNN
+	1    8800 1350
+	1    0    0    -1
+$EndComp
+$Comp
+L power:VCC #PWR?
+U 1 1 6210697E
+P 9050 1250
+F 0 "#PWR?" H 9050 1100 50  0001 C CNN
+F 1 "VCC" H 9065 1423 50  0000 C CNN
+F 2 "" H 9050 1250 50  0001 C CNN
+F 3 "" H 9050 1250 50  0001 C CNN
+	1    9050 1250
+	1    0    0    -1
+$EndComp
+$Comp
+L power:VCC #PWR?
+U 1 1 62106C4A
+P 8800 1250
+F 0 "#PWR?" H 8800 1100 50  0001 C CNN
+F 1 "VCC" H 8815 1423 50  0000 C CNN
+F 2 "" H 8800 1250 50  0001 C CNN
+F 3 "" H 8800 1250 50  0001 C CNN
+	1    8800 1250
+	1    0    0    -1
+$EndComp
+Wire Wire Line
+	9050 1550 9050 1450
+Wire Wire Line
+	8500 1550 9050 1550
+Wire Wire Line
+	8500 1650 8800 1650
+Wire Wire Line
+	8800 1450 8800 1650
+Connection ~ 8800 1650
+Wire Wire Line
+	8800 1650 9400 1650
 $EndSCHEMATC

Commit message: pcb left v1.2
Parts:
- gave numbers to parts that had none: 2
Changed lines of the file:
@@
 SDA
 $Comp
-L Device:R_Small R?
+L Device:R_Small R8
 U 1 1 6210052B
 P 9050 1350
-F 0 "R?" H 9109 1396 50  0000 L CNN
+F 0 "R8" H 9109 1396 50  0000 L CNN
 F 1 "10K" H 9109 1305 50  0000 L CNN
 F 2 "Resistor_SMD:R_0805_2012Metric" H 9050 1350 50  0001 C CNN
@@
 Connection ~ 9050 1550
 $Comp
-L Device:R_Small R?
+L Device:R_Small R7
 U 1 1 621066F7
 P 8800 1350
-F 0 "R?" H 8859 1396 50  0000 L CNN
+F 0 "R7" H 8859 1396 50  0000 L CNN
 F 1 "10K" H 8859 1305 50  0000 L CNN
 F 2 "Resistor_SMD:R_0805_2012Metric" H 8800 1350 50  0001 C CNN
@@
 $EndComp
 $Comp
-L power:VCC #PWR?
+L power:VCC #PWR052
 U 1 1 6210697E
 P 9050 1250
-F 0 "#PWR?" H 9050 1100 50  0001 C CNN
+F 0 "#PWR052" H 9050 1100 50  0001 C CNN
 F 1 "VCC" H 9065 1423 50  0000 C CNN
 F 2 "" H 9050 1250 50  0001 C CNN
@@
 $EndComp
 $Comp
-L power:VCC #PWR?
+L power:VCC #PWR051
 U 1 1 62106C4A
 P 8800 1250
-F 0 "#PWR?" H 8800 1100 50  0001 C CNN
+F 0 "#PWR051" H 8800 1100 50  0001 C CNN
 F 1 "VCC" H 8815 1423 50  0000 C CNN
 F 2 "" H 8800 1250 50  0001 C CNN

Commit message: pcb fixes
Parts:
- removed C1: 10uF, Capacitor_SMD:C_0805_2012Metric, symbol Device:C_Small
- removed C10, C11: 6pF, Capacitor_SMD:C_0805_2012Metric, symbol Device:C_Small
- removed C2, C3, C4, C5, C6, C7: 0.1uF, Capacitor_SMD:C_0805_2012Metric, symbol Device:C_Small
- removed D26: D, Diode_SMD:D_MiniMELF, symbol Device:D_Small
- removed D27: PRTR5V0U2X, Package_TO_SOT_SMD:SOT-143, symbol Power_Protection:PRTR5V0U2X
- removed F1: 500mA, Fuse:Fuse_0805_2012Metric, symbol Device:Polyfuse_Small
- removed J1: AudioJack4, Local:TRRS-PJ-320A, symbol Connector:AudioJack4
- removed J2: AVR-ISP-6, Local:AVR-ISP-6, symbol Connector:AVR-ISP-6
- removed R1, R7, R8: 10K, Resistor_SMD:R_0805_2012Metric, symbol Device:R_Small
- removed R3, R4: 5.1K, Resistor_SMD:R_0805_2012Metric, symbol Device:R_Small
- removed R5, R6: 22, Resistor_SMD:R_0805_2012Metric, symbol Device:R_Small
- removed SW26: SW_Push, Local:LL3301NF065QG, symbol Switch:SW_Push
- removed USB1: HRO-TYPE-C-31-M-12, Type-C:HRO-TYPE-C-31-M-12, symbol Type-C:HRO-TYPE-C-31-M-12
- removed Y1: 16MHz, Crystal:Crystal_SMD_3225-4Pin_3.2x2.5mm, symbol Device:Crystal_GND24_Small
Connections:
- no-connect marks 3 -> 7
Other:
- moved on the sheet: C8, R2, U1
